File: KiCAD/PrawnBlaster_Connectorized.kicad_pcb (KiCad board)
At the start: 2 copper layers, 93 x 58.4 mm, 37 parts, among them IC1 74LVT245D,118, J1 PWR SEL, J2 Ext. Clock, J3 Ext. Trig., J4 Pseudoclock 3, J5 Pseudoclock 1, J6 Pseudoclock 2, J7 Pseudoclock 0, J8 EXT PWR, U2 74LVC1G34, U3 Pico, U4 74LVC1G17

Commit message: 3D Models Update 2
Parts:
- R3, R4, R5, R6, R7, R9: footprint Resistor_SMD:R_1206_3216Metric_Pad1.30x1.75mm_HandSolder -> Resistor_SMD:R_0805_2012Metric_Pad1.20x1.40mm_HandSolder
